File: aaLogger.sch (EAGLE design)
At the start: 55 parts, among them Q1 IRLML6244TR, U1 MCP1640C, U2 ATmega328P-AU

Commit message: Near final.
Parts:
- added C10, C9: 27pF, _jc:C-USM0805
- added C11, C13: 100nF, _jc:C-USM0805
- added JMP1: solder jumper, _jc:R-US_M0805
- added JP3: GNDSEL, SparkFun:M03LOCK
- added JP4: RTC BACKUP, SparkFun:M03LOCK
- added LOGO1, LOGO2: OSHW_LOGO_8MILX0150-NT, ohw-logo:OSHW_LOGO_8MILX0150-NT
- added PR13: PROTO-3, _jc:PROTO-3
- B1: value (none) -> CR2016
- C1: value 100nF -> 10uF; device _jc:C-USC0805 -> _jc:C-USM0805
- C12, C4, C5, C6, C7, C8: device _jc:C-USC0805 -> _jc:C-USM0805
- J1: value (none) -> ICSP
- L1: device _jc:INDUCTORR1210 -> _jc:INDUCTORNRS5020
- PR1, PR10, PR11, PR12, PR2, PR3, PR4, PR5, PR6, PR7, PR8, PR9: value PROTO-5 -> PROTO-10; device _jc:PROTO-5 -> _jc:PROTO-10
- R10: value 249K -> 2.2K
- R11: value solder jumper -> 10K
- R12: value 100 -> 220
- R3: value 47.5K -> 249K
- R4: value 10K -> 47.5K
- R5: value 2.2K -> 10K
- R6: device _jc:R-US_R0805 -> _jc:R-US_M0805
- S1: value (none) -> RESET
- S2: value (none) -> START/INIT
- S3: value (none) -> DL/SET
- TB1: value 3 - 4.5VDC -> +BAT-
- U3: value (none) -> DS3232
- U4, U5: value (none) -> M24M02
- Y1: value (none) -> 8MHz; device _jc:RESONATORZTT -> _jc:RESONATOR
Connections:
- removed net /WC: U2.PD2(INT0), U4./WC, U5./WC
- removed net PGND: Q1.D, U$2.PIN01, U$2.PIN02, U$2.PIN03, U$2.PIN04, U$2.PIN05, U$2.PIN06, U$2.PIN07, U$2.PIN08, U$2.PIN09, U$2.PIN10, U$2.PIN11, U$2.PIN12, U3.GND, U3.NC1, U3.NC10, U3.NC11, U3.NC12, U3.NC13, U3.NC14, U3.NC19, U3.NC2, U3.NC7, U3.NC8, U3.NC9, U4.E2, U4.GND, U5.GND
- new net N$10: PR3.10, PR3.6, PR3.7, PR3.8, PR3.9
- new net N$14: PR4.10, PR4.6, PR4.7, PR4.8, PR4.9
- new net N$15: PR6.10, PR6.6, PR6.7, PR6.8, PR6.9
- new net N$28: PR7.10, PR7.6, PR7.7, PR7.8, PR7.9
- new net N$30: PR8.10, PR8.6, PR8.7, PR8.8, PR8.9
- new net N$31: PR9.10, PR9.6, PR9.7, PR9.8, PR9.9
- new net N$32: PR10.10, PR10.6, PR10.7, PR10.8, PR10.9
- new net N$33: PR11.10, PR11.6, PR11.7, PR11.8, PR11.9
- new net N$34: PR12.10, PR12.6, PR12.7, PR12.8, PR12.9
- new net N$35: JP4.2, U3.VBAT
- new net N$36: JP3.1, Q1.D
- new net N$4: PR1.10, PR1.6, PR1.7, PR1.8, PR1.9
- new net N$5: PR5.10, PR5.6, PR5.7, PR5.8, PR5.9
- new net N$9: PR2.10, PR2.6, PR2.7, PR2.8, PR2.9
- new net SGND: JP3.2, U$2.1, U$2.10, U$2.11, U$2.12, U$2.2, U$2.3, U$2.4, U$2.5, U$2.6, U$2.7, U$2.8, U$2.9
- new net SPWR: R12.2, U2.PB1(OC1A)
- net /RESET: now also C5.1; no longer C12.1
- net 32KHZ: now also R11.1
- net ADC6: now also C4.2, R5.2; no longer R4.2
- net ADC7: now also C4.1, R4.2, R5.1; no longer R3.2, R4.1
- net BAT: now also C1.1, JP4.1, R4.1; no longer C2.1, R3.1
- net GND: now also B1.B-, C10.2, C11.2, C12.2, C13.2, C9.2, JMP1.2, JP3.3, PR13.1, PR13.2, PR13.3, R3.2, U3.GND, U3.NC1, U3.NC10, U3.NC11, U3.NC12, U3.NC13, U3.NC14, U3.NC19, U3.NC2, U3.NC7, U3.NC8, U3.NC9, U4./WC, U4.E2, U4.GND, U5./WC, U5.GND; no longer B1.NEG, C4.2, C5.2, R10.2, R11.2
- net LED1: now also R7.2; no longer R5.2
- net LED2: now also R8.2; no longer R7.2
- net MISO: now also JP1.11; no longer JP1.10
- net MOSI: now also JP1.12; no longer JP1.11
- net N$1: now also JP4.3; no longer U3.VBAT
- net N$11: now also C10.1
- net N$12: now also JMP1.1, R3.1; no longer R10.1, R11.1
- net N$13: now also C8.1; no longer C5.1
- net N$2: now also R7.1; no longer R5.1
- net N$3: now also R8.1; no longer R7.1
- net N$8: now also C9.1
- net PPWR: now also C11.1, C12.1, C13.1, U2.PD2(INT0), U3.VCC, U4.VCC, U5.E2, U5.VCC; no longer R12.2, U2.PB1(OC1A)
- net RST: now also C5.2; no longer C12.2
- net SCK: now also JP1.10; no longer JP1.12
- net SCL: now also R10.1; no longer R9.1
- net SDA: now also R9.1; no longer R8.1
- net SW2: now also U2.PD6(AIN0); no longer U2.PD5(T1)
- net SW3: now also U2.PD5(T1); no longer U2.PD6(AIN0)
- net VCC: now also C2.1, R10.2, R11.2, U$1.1, U$1.10, U$1.11, U$1.12, U$1.2, U$1.3, U$1.4, U$1.5, U$1.6, U$1.7, U$1.8, U$1.9; no longer C1.1, C4.1, C8.1, R8.2, U$1.PIN01, U$1.PIN02, U$1.PIN03, U$1.PIN04, U$1.PIN05, U$1.PIN06, U$1.PIN07, U$1.PIN08, U$1.PIN09, U$1.PIN10, U$1.PIN11, U$1.PIN12, U3.VCC, U4.VCC, U5.E2, U5.VCC
Other:
- moved on the sheet: B1, C1, C12, C2, C3, C4, C5, C6, C7, C8, D1, D2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

Commit message: v1 as sent to iTead.
Parts:
- JP1: value M12PTH -> PROTO-12NR; device SparkFun:M12PTH -> _jc:PROTO-12NR
- R7, R8: value 2.2K -> 1K
- U$1, U$2: value PROTO-12 -> PROTO-12PROTO; device _jc:PROTO-12 -> _jc:PROTO-12PROTO
Other:
- note added: "Double-A DataLogger"
- note added: "by Jack Christensen CC BY-SA"
- note added: "v1"
Changed lines of the file:
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@@
 <part name="U5" library="_jc" deviceset="M24M02" device="" value="M24M02"/>
 <part name="GND2" library="supply1" deviceset="GND" device=""/>
-<part name="R7" library="_jc" deviceset="R-US_" device="M0805" value="2.2K"/>
-<part name="R8" library="_jc" deviceset="R-US_" device="M0805" value="2.2K"/>
+<part name="R7" library="_jc" deviceset="R-US_" device="M0805" value="1K"/>
+<part name="R8" library="_jc" deviceset="R-US_" device="M0805" value="1K"/>
 <part name="GND5" library="supply1" deviceset="GND" device=""/>
 <part name="GND7" library="supply1" deviceset="GND" device=""/>
@@
 <part name="PR6" library="_jc" deviceset="PROTO-10" device=""/>
 <part name="PR7" library="_jc" deviceset="PROTO-10" device=""/>
-<part name="JP1" library="SparkFun" deviceset="M12" device="PTH"/>
+<part name="JP1" library="_jc" deviceset="PROTO-12" device="NR"/>
 <part name="PR1" library="_jc" deviceset="PROTO-10" device=""/>
 <part name="PR5" library="_jc" deviceset="PROTO-10" device=""/>
@@
 <part name="PR11" library="_jc" deviceset="PROTO-10" device=""/>
 <part name="PR12" library="_jc" deviceset="PROTO-10" device=""/>
-<part name="U$1" library="_jc" deviceset="PROTO-12" device=""/>
-<part name="U$2" library="_jc" deviceset="PROTO-12" device=""/>
+<part name="U$1" library="_jc" deviceset="PROTO-12" device="PROTO" value="PROTO-12PROTO"/>
+<part name="U$2" library="_jc" deviceset="PROTO-12" device="PROTO" value="PROTO-12PROTO"/>
 <part name="P+6" library="supply1" deviceset="VCC" device=""/>
 <part name="Q1" library="_jc" deviceset="MOSFET-NCHANNEL" device="SOT23" value="IRLML6244TR"/>
@@
 <sheet>
 <plain>
+<text x="149.86" y="30.48" size="3.81" layer="94" ratio="12">Double-A DataLogger</text>
+<text x="149.86" y="25.4" size="2.54" layer="94" ratio="12">by Jack Christensen CC BY-SA</text>
+<text x="236.22" y="7.62" size="2.54" layer="94" ratio="12">v1</text>
 </plain>
 <instances>
@@
 <instance part="PR6" gate="G$1" x="223.52" y="170.18"/>
 <instance part="PR7" gate="G$1" x="223.52" y="167.64"/>
-<instance part="JP1" gate="G$1" x="109.22" y="160.02" rot="R180"/>
+<instance part="JP1" gate="G$1" x="246.38" y="119.38" rot="R270"/>
 <instance part="PR1" gate="G$1" x="223.52" y="182.88"/>
 <instance part="PR5" gate="G$1" x="223.52" y="172.72"/>
@@
 <instance part="PR13" gate="G$1" x="195.58" y="167.64" rot="R90"/>
 <instance part="B1" gate="G$1" x="220.98" y="48.26" rot="MR0"/>
-<instance part="JP3" gate="G$1" x="116.84" y="172.72"/>
+<instance part="JP3" gate="G$1" x="116.84" y="172.72" smashed="yes">
+<attribute name="VALUE" x="113.284" y="167.894" size="1.778" layer="96" rot="R90"/>
+<attribute name="NAME" x="114.3" y="178.562" size="1.778" layer="95"/>
+</instance>
 <instance part="GND20" gate="1" x="127" y="175.26" smashed="yes" rot="R90">
 <attribute name="VALUE" x="129.54" y="172.72" size="1.778" layer="96" rot="R90"/>
@@
 <segment>
 <pinref part="JP1" gate="G$1" pin="8"/>
-<wire x1="99.06" y1="157.48" x2="91.44" y2="157.48" width="0.1524" layer="91"/>
-<label x="91.44" y="157.48" size="1.778" layer="95"/>
+<wire x1="246.38" y1="111.76" x2="236.22" y2="111.76" width="0.1524" layer="91"/>
+<label x="236.22" y="111.76" size="1.778" layer="95"/>
 </segment>
 </net>
@@
 <segment>
 <pinref part="JP1" gate="G$1" pin="2"/>
-<wire x1="99.06" y1="172.72" x2="91.44" y2="172.72" width="0.1524" layer="91"/>
-<label x="91.44" y="172.72" size="1.778" layer="95"/>
+<wire x1="246.38" y1="142.24" x2="236.22" y2="142.24" width="0.1524" layer="91"/>
+<label x="236.22" y="142.24" size="1.778" layer="95"/>
 </segment>
 </net>
@@
 <segment>
 <pinref part="JP1" gate="G$1" pin="3"/>
-<wire x1="99.06" y1="170.18" x2="91.44" y2="170.18" width="0.1524" layer="91"/>
-<label x="91.44" y="170.18" size="1.778" layer="95"/>
+<wire x1="246.38" y1="137.16" x2="236.22" y2="137.16" width="0.1524" layer="91"/>
+<label x="236.22" y="137.16" size="1.778" layer="95"/>
 </segment>
 </net>
@@
 <segment>
 <pinref part="JP1" gate="G$1" pin="10"/>
-<wire x1="99.06" y1="152.4" x2="91.44" y2="152.4" width="0.1524" layer="91"/>
-<label x="91.44" y="152.4" size="1.778" layer="95"/>
+<wire x1="246.38" y1="101.6" x2="236.22" y2="101.6" width="0.1524" layer="91"/>
+<label x="236.22" y="101.6" size="1.778" layer="95"/>
 </segment>
 </net>
@@
 <segment>
 <pinref part="JP1" gate="G$1" pin="11"/>
-<wire x1="99.06" y1="149.86" x2="91.44" y2="149.86" width="0.1524" layer="91"/>
-<label x="91.44" y="149.86" size="1.778" layer="95"/>
+<wire x1="246.38" y1="96.52" x2="236.22" y2="96.52" width="0.1524" layer="91"/>
+<label x="236.22" y="96.52" size="1.778" layer="95"/>
 </segment>
 </net>
@@
 <segment>
 <pinref part="JP1" gate="G$1" pin="12"/>
-<wire x1="99.06" y1="147.32" x2="91.44" y2="147.32" width="0.1524" layer="91"/>
-<label x="91.44" y="147.32" size="1.778" layer="95"/>
+<wire x1="246.38" y1="91.44" x2="236.22" y2="91.44" width="0.1524" layer="91"/>
+<label x="236.22" y="91.44" size="1.778" layer="95"/>
 </segment>
 </net>
@@
 <segment>
 <pinref part="JP1" gate="G$1" pin="1"/>
-<wire x1="99.06" y1="175.26" x2="91.44" y2="175.26" width="0.1524" layer="91"/>
-<label x="91.44" y="175.26" size="1.778" layer="95"/>
+<wire x1="246.38" y1="147.32" x2="236.22" y2="147.32" width="0.1524" layer="91"/>
+<label x="236.22" y="147.32" size="1.778" layer="95"/>
 </segment>
 </net>
@@
 <segment>
 <pinref part="JP1" gate="G$1" pin="4"/>
-<wire x1="99.06" y1="167.64" x2="91.44" y2="167.64" width="0.1524" layer="91"/>
-<label x="91.44" y="167.64" size="1.778" layer="95"/>
+<wire x1="246.38" y1="132.08" x2="236.22" y2="132.08" width="0.1524" layer="91"/>
+<label x="236.22" y="132.08" size="1.778" layer="95"/>
 </segment>
 </net>
@@
 <segment>
 <pinref part="JP1" gate="G$1" pin="5"/>
-<wire x1="99.06" y1="165.1" x2="91.44" y2="165.1" width="0.1524" layer="91"/>
-<label x="91.44" y="165.1" size="1.778" layer="95"/>
+<wire x1="246.38" y1="127" x2="236.22" y2="127" width="0.1524" layer="91"/>
+<label x="236.22" y="127" size="1.778" layer="95"/>
 </segment>
 </net>
@@
 <segment>
 <pinref part="JP1" gate="G$1" pin="6"/>
-<wire x1="99.06" y1="162.56" x2="91.44" y2="162.56" width="0.1524" layer="91"/>
-<label x="91.44" y="162.56" size="1.778" layer="95"/>
+<wire x1="246.38" y1="121.92" x2="236.22" y2="121.92" width="0.1524" layer="91"/>
+<label x="236.22" y="121.92" size="1.778" layer="95"/>
 </segment>
 </net>
@@
 <segment>
 <pinref part="JP1" gate="G$1" pin="7"/>
-<wire x1="99.06" y1="160.02" x2="91.44" y2="160.02" width="0.1524" layer="91"/>
-<label x="91.44" y="160.02" size="1.778" layer="95"/>
+<wire x1="246.38" y1="116.84" x2="236.22" y2="116.84" width="0.1524" layer="91"/>
+<label x="236.22" y="116.84" size="1.778" layer="95"/>
 </segment>
 </net>
@@
 <segment>
 <pinref part="JP1" gate="G$1" pin="9"/>
-<wire x1="99.06" y1="154.94" x2="91.44" y2="154.94" width="0.1524" layer="91"/>
-<label x="91.44" y="154.94" size="1.778" layer="95"/>
-</segment>
-</net>
+<wire x1="246.38" y1="106.68" x2="236.22" y2="106.68" width="0.1524" layer="91"/>
+<label x="236.22" y="106.68" size="1.778" layer="95"/>
+</segment>
+</net>

Commit message: Remove R11, not needed. Reroute 32K, move RTC slightly.
Parts:
- removed R11: 10K, _jc:R-US_M0805
Connections:
- net 32KHZ: no longer R11.1
- net VCC: no longer R11.2
Other:
- note added: "v2"
- note removed: "v1"
- moved on the sheet: U4, U5
Changed lines of the file:
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@@
 <part name="D1" library="adafruit" deviceset="LED" device="CHIPLED_1206" value="Red"/>
 <part name="D2" library="adafruit" deviceset="LED" device="CHIPLED_1206" value="Green"/>
-<part name="U4" library="_jc" deviceset="M24M02" device="" value="M24M02"/>
+<part name="U5" library="_jc" deviceset="M24M02" device="" value="M24M02"/>
 <part name="U3" library="_jc" deviceset="DS3232" device="" value="DS3232"/>
 <part name="U1" library="_jc" deviceset="MCP1640" device="" value="MCP1640C"/>
@@
 <part name="R4" library="_jc" deviceset="R-US_" device="M0805" value="47.5K"/>
 <part name="R5" library="_jc" deviceset="R-US_" device="M0805" value="10K"/>
-<part name="U5" library="_jc" deviceset="M24M02" device="" value="M24M02"/>
+<part name="U4" library="_jc" deviceset="M24M02" device="" value="M24M02"/>
 <part name="GND2" library="supply1" deviceset="GND" device=""/>
 <part name="R7" library="_jc" deviceset="R-US_" device="M0805" value="1K"/>
@@
 <part name="R13" library="_jc" deviceset="R-US_" device="M0805" value="10K"/>
 <part name="GND11" library="supply1" deviceset="GND" device=""/>
-<part name="R11" library="_jc" deviceset="R-US_" device="M0805" value="10K"/>
-<part name="P+9" library="supply1" deviceset="VCC" device=""/>
 <part name="C4" library="_jc" deviceset="C-US" device="M0805" value="100nF"/>
 <part name="GND16" library="supply1" deviceset="GND" device=""/>
@@
 <text x="149.86" y="30.48" size="3.81" layer="94" ratio="12">Double-A DataLogger</text>
 <text x="149.86" y="25.4" size="2.54" layer="94" ratio="12">by Jack Christensen CC BY-SA</text>
-<text x="236.22" y="7.62" size="2.54" layer="94" ratio="12">v1</text>
+<text x="236.22" y="7.62" size="2.54" layer="94" ratio="12">v2</text>
 </plain>
 <instances>
@@
 <instance part="D1" gate="G$1" x="5.08" y="66.04"/>
 <instance part="D2" gate="G$1" x="15.24" y="66.04"/>
-<instance part="U4" gate="G$1" x="182.88" y="101.6"/>
+<instance part="U5" gate="G$1" x="182.88" y="101.6"/>
 <instance part="U3" gate="G$1" x="185.42" y="66.04"/>
 <instance part="U1" gate="G$1" x="63.5" y="25.4" smashed="yes">
@@
 <attribute name="VALUE" x="22.098" y="24.13" size="1.778" layer="96" rot="R270"/>
 </instance>
-<instance part="U5" gate="G$1" x="182.88" y="124.46"/>
+<instance part="U4" gate="G$1" x="182.88" y="124.46"/>
 <instance part="GND2" gate="1" x="10.16" y="55.88" smashed="yes">
 <attribute name="VALUE" x="7.62" y="53.34" size="1.778" layer="96"/>
@@
 <attribute name="VALUE" x="129.54" y="149.86" size="1.778" layer="96"/>
 </instance>
-<instance part="R11" gate="G$1" x="218.44" y="68.58" smashed="yes" rot="R90">
-<attribute name="NAME" x="221.7674" y="62.992" size="1.778" layer="95" rot="R90"/>
-<attribute name="VALUE" x="221.742" y="69.85" size="1.778" layer="96" rot="R90"/>
-</instance>
-<instance part="P+9" gate="VCC" x="218.44" y="81.28"/>
 <instance part="C4" gate="G$1" x="30.48" y="20.32"/>
 <instance part="GND16" gate="1" x="165.1" y="43.18" smashed="yes">
@@
 <junction x="180.34" y="182.88"/>
 <junction x="175.26" y="182.88"/>
-</segment>
-<segment>
-<pinref part="R11" gate="G$1" pin="2"/>
-<wire x1="218.44" y1="73.66" x2="218.44" y2="78.74" width="0.1524" layer="91"/>
-<pinref part="P+9" gate="VCC" pin="VCC"/>
 </segment>
 </net>
@@
 <pinref part="U3" gate="G$1" pin="GND"/>
 <wire x1="167.64" y1="50.8" x2="165.1" y2="50.8" width="0.1524" layer="91"/>
+<pinref part="U5" gate="G$1" pin="GND"/>
+<wire x1="167.64" y1="96.52" x2="165.1" y2="96.52" width="0.1524" layer="91"/>
+<junction x="165.1" y="78.74"/>
 <pinref part="U4" gate="G$1" pin="GND"/>
-<wire x1="167.64" y1="96.52" x2="165.1" y2="96.52" width="0.1524" layer="91"/>
-<wire x1="165.1" y1="96.52" x2="165.1" y2="91.44" width="0.1524" layer="91"/>
-<junction x="165.1" y="78.74"/>
-<pinref part="U5" gate="G$1" pin="GND"/>
-<wire x1="165.1" y1="91.44" x2="165.1" y2="78.74" width="0.1524" layer="91"/>
+<wire x1="165.1" y1="96.52" x2="165.1" y2="78.74" width="0.1524" layer="91"/>
 <wire x1="167.64" y1="119.38" x2="165.1" y2="119.38" width="0.1524" layer="91"/>
+<junction x="165.1" y="96.52"/>
 <wire x1="165.1" y1="119.38" x2="165.1" y2="96.52" width="0.1524" layer="91"/>
-<junction x="165.1" y="96.52"/>
-<pinref part="U4" gate="G$1" pin="E2"/>
-<wire x1="198.12" y1="99.06" x2="200.66" y2="99.06" width="0.1524" layer="91"/>
-<wire x1="200.66" y1="99.06" x2="200.66" y2="91.44" width="0.1524" layer="91"/>
-<wire x1="200.66" y1="91.44" x2="165.1" y2="91.44" width="0.1524" layer="91"/>
-<junction x="165.1" y="91.44"/>
 <pinref part="GND16" gate="1" pin="GND"/>
 <wire x1="165.1" y1="45.72" x2="165.1" y2="50.8" width="0.1524" layer="91"/>
@@
 </segment>
 <segment>
-<pinref part="U4" gate="G$1" pin="/WC"/>
+<pinref part="U5" gate="G$1" pin="/WC"/>
 <wire x1="198.12" y1="96.52" x2="210.82" y2="96.52" width="0.1524" layer="91"/>
 <wire x1="210.82" y1="96.52" x2="210.82" y2="119.38" width="0.1524" layer="91"/>
-<pinref part="U5" gate="G$1" pin="/WC"/>
-<wire x1="210.82" y1="119.38" x2="198.12" y2="119.38" width="0.1524" layer="91"/>
+<pinref part="U4" gate="G$1" pin="/WC"/>
+<wire x1="210.82" y1="119.38" x2="200.66" y2="119.38" width="0.1524" layer="91"/>
 <pinref part="GND17" gate="1" pin="GND"/>
+<wire x1="200.66" y1="119.38" x2="198.12" y2="119.38" width="0.1524" layer="91"/>
 <wire x1="210.82" y1="96.52" x2="210.82" y2="93.98" width="0.1524" layer="91"/>
 <junction x="210.82" y="96.52"/>
+<pinref part="U4" gate="G$1" pin="E2"/>
+<wire x1="198.12" y1="121.92" x2="200.66" y2="121.92" width="0.1524" layer="91"/>
+<wire x1="200.66" y1="121.92" x2="200.66" y2="119.38" width="0.1524" layer="91"/>
+<junction x="200.66" y="119.38"/>
 </segment>
 <segment>
@@
 </segment>
 <segment>
-<pinref part="U5" gate="G$1" pin="SCL"/>
+<pinref part="U4" gate="G$1" pin="SCL"/>
 <wire x1="198.12" y1="127" x2="208.28" y2="127" width="0.1524" layer="91"/>
 <label x="203.2" y="127" size="1.778" layer="95"/>
 </segment>
 <segment>
-<pinref part="U4" gate="G$1" pin="SCL"/>
+<pinref part="U5" gate="G$1" pin="SCL"/>
 <wire x1="198.12" y1="104.14" x2="208.28" y2="104.14" width="0.1524" layer="91"/>
 <label x="203.2" y="104.14" size="1.778" layer="95"/>
@@
 </segment>
 <segment>
-<pinref part="U5" gate="G$1" pin="SDA"/>
+<pinref part="U4" gate="G$1" pin="SDA"/>
 <wire x1="198.12" y1="124.46" x2="208.28" y2="124.46" width="0.1524" layer="91"/>
 <label x="203.2" y="124.46" size="1.778" layer="95"/>
 </segment>
 <segment>
-<pinref part="U4" gate="G$1" pin="SDA"/>
+<pinref part="U5" gate="G$1" pin="SDA"/>
 <wire x1="198.12" y1="101.6" x2="208.28" y2="101.6" width="0.1524" layer="91"/>
 <label x="203.2" y="101.6" size="1.778" layer="95"/>
@@
 <wire x1="203.2" y1="60.96" x2="218.44" y2="60.96" width="0.1524" layer="91"/>
 <label x="208.28" y="60.96" size="1.778" layer="95"/>
-<pinref part="R11" gate="G$1" pin="1"/>
-<wire x1="218.44" y1="60.96" x2="218.44" y2="63.5" width="0.1524" layer="91"/>
 </segment>
 <segment>
@@
 <net name="PPWR" class="0">
 <segment>
-<pinref part="U5" gate="G$1" pin="VCC"/>
+<pinref part="U4" gate="G$1" pin="VCC"/>
 <pinref part="C13" gate="G$1" pin="1"/>
 <wire x1="167.64" y1="127" x2="162.56" y2="127" width="0.1524" layer="91"/>
 <wire x1="162.56" y1="127" x2="157.48" y2="127" width="0.1524" layer="91"/>
 <wire x1="157.48" y1="127" x2="157.48" y2="124.46" width="0.1524" layer="91"/>
-<pinref part="U5" gate="G$1" pin="E2"/>
-<wire x1="198.12" y1="121.92" x2="200.66" y2="121.92" width="0.1524" layer="91"/>
-<wire x1="200.66" y1="121.92" x2="200.66" y2="134.62" width="0.1524" layer="91"/>
-<wire x1="200.66" y1="134.62" x2="162.56" y2="134.62" width="0.1524" layer="91"/>
 <wire x1="162.56" y1="134.62" x2="162.56" y2="127" width="0.1524" layer="91"/>
 <junction x="162.56" y="127"/>
 <wire x1="162.56" y1="134.62" x2="154.94" y2="134.62" width="0.1524" layer="91"/>
-<junction x="162.56" y="134.62"/>
-<pinref part="U4" gate="G$1" pin="VCC"/>
+<pinref part="U5" gate="G$1" pin="VCC"/>
 <pinref part="C12" gate="G$1" pin="1"/>
 <wire x1="167.64" y1="104.14" x2="162.56" y2="104.14" width="0.1524" layer="91"/>
 <wire x1="162.56" y1="104.14" x2="157.48" y2="104.14" width="0.1524" layer="91"/>
 <wire x1="157.48" y1="104.14" x2="157.48" y2="101.6" width="0.1524" layer="91"/>
-<wire x1="162.56" y1="127" x2="162.56" y2="104.14" width="0.1524" layer="91"/>
+<wire x1="162.56" y1="127" x2="162.56" y2="111.76" width="0.1524" layer="91"/>
 <junction x="162.56" y="104.14"/>
 <pinref part="U3" gate="G$1" pin="VCC"/>
 <pinref part="C11" gate="G$1" pin="1"/>
+<wire x1="162.56" y1="111.76" x2="162.56" y2="104.14" width="0.1524" layer="91"/>
 <wire x1="167.64" y1="81.28" x2="162.56" y2="81.28" width="0.1524" layer="91"/>
 <wire x1="162.56" y1="81.28" x2="157.48" y2="81.28" width="0.1524" layer="91"/>
@@
 <junction x="162.56" y="81.28"/>
 <label x="154.94" y="134.62" size="1.778" layer="95"/>
-</segment>
-<segment>
+<pinref part="U5" gate="G$1" pin="E2"/>
+<wire x1="198.12" y1="99.06" x2="200.66" y2="99.06" width="0.1524" layer="91"/>
+<wire x1="200.66" y1="99.06" x2="200.66" y2="111.76" width="0.1524" layer="91"/>
+<wire x1="200.66" y1="111.76" x2="162.56" y2="111.76" width="0.1524" layer="91"/>
+<junction x="162.56" y="111.76"/>
+</segment>
+<segment>
